File: V2.sch (EAGLE design)
At the start: 51 parts, among them IC1 LM2596S, U1 BTS7960B, U2 BTS7960B, U3 BTS7960B, U4 BTS7960B, U5 SN74AHC244DW, U6 MCP2551

Commit message: V2 finished
Other:
- note added: "DC/DC COVERTER"
- note removed: "DC/DC COVERTERS"
Changed lines of the file:
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@@
 <text x="89.662" y="4.064" size="5.08" layer="97">MCU</text>
 <text x="185.42" y="170.18" size="5.08" layer="97">CAN  </text>
-<text x="114.046" y="173.482" size="5.08" layer="97">DC/DC COVERTERS</text>
-<text x="60.198" y="174.244" size="5.08" layer="97">GPIO</text>
+<text x="114.046" y="173.482" size="5.08" layer="97">DC/DC COVERTER</text>
+<text x="57.658" y="174.244" size="5.08" layer="97">GPIO</text>
 <text x="81.28" y="127" size="5.08" layer="97">MOTOR DRIVERS UNIT</text>
 <wire x1="76.2" y1="55.88" x2="106.68" y2="55.88" width="0.1524" layer="97" style="shortdash"/>
